File: schematic/r68.kicad_pcb (KiCad board)
At the start: 2 copper layers, 285.8 x 95.3 mm, 146 parts, among them K0 K_ESC, K0A1 K_0, K0B1 K_MIN, K0C1 K_EQL, K0D1 K_BS, K1 K_1, K10 K_TAB, K11 K_Q, K12 K_W, K13 K_E, K14 K_R, K15 K_T, K16 K_Y, K17 K_U, K18 K_I, K19 K_O, K1A1 K_P, K1B1 K_OBR, K1C1 K_CBR, K1D1 K_BSL, K2 K_2, K20 K_CAP, K21 K_A, K22 K_S, K23 K_D, K24 K_F, K25 K_G, K26 K_H, K27 K_J, K28 K_K, K29 K_L, K2A1 K_COL, K2B1 K_QOT, K2C1 K_ENT, K3 K_3, K30 K_LSH, K31 K_Z, K32 K_X, K33 K_C, K34 K_V, K35 K_B, K36 K_N, K37 K_M, K38 K_COM, K39 K_DOT, K3A1 K_QUE, K3B1 K_RSH, K4 K_4, K40 K_LCL, K41 K_LWN, K42 K_LAL, K45 K_SP, K48 K_RFN, K49 K_RALT, K4A1 K_RWIN, K4B1 K_RCTL, K5 K_5, K6 K_6, K7 K_7, K8 K_8, K9 K_9, P1 USB_B, P2 SPKR, SW1 SW_Push, U1 ATmega32U4-AU, Y1 16MHz

Commit message: route for 68 key
Parts:
- removed D4B1: D, Diodes_SMD:D_SOD-323
- removed G***: LOGO, logos:ron-test
- removed K4B1: K_RCTL, Keyboard:CHERRY_PCB_125H
- removed REF** (x4): , Mounting_Holes:MountingHole_2.7mm_M2.5
- added D0D2: D, Diodes_SMD:D_SOD-323, B.Cu at (324.9, 58.3)
- added D0D3: D, Diodes_SMD:D_SOD-323, B.Cu at (324.9, 77.4)
- added D0D4: D, Diodes_SMD:D_SOD-323, B.Cu at (324.9, 96.4)
- added D0D5: D, Diodes_SMD:D_SOD-323, B.Cu at (305.9, 115.5)
- added D0D6: D, Diodes_SMD:D_SOD-323, B.Cu at (324.9, 115.5)
- added D0D7: D, Diodes_SMD:D_SOD-323, B.Cu at (286.8, 134.5)
- added D0D8: D, Diodes_SMD:D_SOD-323, B.Cu at (305.9, 134.5)
- added D0D9: D, Diodes_SMD:D_SOD-323, B.Cu at (325.0, 134.5)
- added K0D2: K_HOME, Keyboard:CHERRY_PCB_100H, F.Cu at (323.9, 52.4)
- added K0D3: K_END, Keyboard:CHERRY_PCB_100H, F.Cu at (323.9, 71.4)
- added K0D4: K_PGUP, Keyboard:CHERRY_PCB_100H, F.Cu at (323.9, 90.5)
- added K0D5: K_UP, Keyboard:CHERRY_PCB_100H, F.Cu at (304.8, 109.5)
- added K0D6: K_PGDN, Keyboard:CHERRY_PCB_100H, F.Cu at (323.9, 109.5)
- added K0D7: K_LEFT, Keyboard:CHERRY_PCB_100H, F.Cu at (285.8, 128.6)
- added K0D8: K_DOWN, Keyboard:CHERRY_PCB_100H, F.Cu at (304.8, 128.6)
- added K0D9: K_RGHT, Keyboard:CHERRY_PCB_100H, F.Cu at (323.9, 128.6)
- added K46: K_FNC, Keyboard:CHERRY_PCB_100H, F.Cu at (228.6, 128.6)
- added K47: K_FN2C, Keyboard:CHERRY_PCB_100H, F.Cu at (247.7, 128.6)
- K3B1: footprint Keyboard:CHERRY_PCB_275H -> Keyboard:CHERRY_PCB_175H
- K48: value K_RFN -> K_FNA
- K49: value K_RALT -> K_FN2A
- K4A1: footprint Keyboard:CHERRY_PCB_125H -> Keyboard:CHERRY_PCB_100H
- moved D4A1 11.9 mm to (267.9, 134.5)
- moved K4A1 11.9 mm to (266.7, 128.6)
- moved K3B1 9.53 mm to (278.6, 109.5)
- moved D3B1 9.52 mm to (279.8, 115.5)
Connections:
- U1 pad 1: (no net) -> /C14
Routing:
- net /C14: track 0.00 -> 288.5 mm, vias 0 -> 1
- net /R3: track 245.8 -> 317.8 mm
- net GND: track 77.3 -> 129.2 mm
- net /C11: track 274.7 -> 225.1 mm, vias 2 -> 1
- net /C13: track 236.2 -> 274.8 mm
- net /R2: track 305.5 -> 338.6 mm
- net /R0: track 352.1 -> 381.9 mm
- net /R1: track 332.0 -> 356.6 mm
- net /C12: track 233.1 -> 249.6 mm
- net /C10: track 230.4 -> 221.5 mm
- net /C8: track 181.8 -> 190.3 mm
- net Net-(D49-Pad2): track 3.32 -> 10.5 mm
- net /C9: track 204.1 -> 211.3 mm
- net VCC: track 212.4 -> 207.7 mm
- net Net-(D0D9-Pad2): track 0.00 -> 3.32 mm
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Other:
- board size 285.8 x 95.3 mm -> 304.8 x 95.3 mm

Commit message: final hole placement and routing
Parts:
- added G***: LOGO, logos:ron-test, B.Cu at (199.6, 86.4)
- added REF**: 1pin, Connectors:1pin, F.Cu at (295.3, 128.6)
- added REF**: 1pin, Connectors:1pin, F.Cu at (289.0, 71.1)
- added REF**: 1pin, Connectors:1pin, F.Cu at (216.2, 128.6)
- added REF**: 1pin, Connectors:1pin, F.Cu at (157.2, 90.5)
- added REF**: 1pin, Connectors:1pin, F.Cu at (54.2, 128.6)
- added REF**: 1pin, Connectors:1pin, F.Cu at (54.2, 71.1)
- moved P1 0.65 mm to (47.0, 47.0)
Routing:
- net /C11: track 225.1 -> 221.1 mm
- net GND: track 129.2 -> 133.1 mm
- net /C0: track 176.7 -> 179.2 mm
- net VCC: track 207.7 -> 207.0 mm
- net /C8: track 190.3 -> 189.6 mm
Other:
- board text added: "It Wrong"
- board text added: "You're Doing"
- board text added: "github.com/rpedde/r68"
- board text added: "http://github.com/rpedde/r68"
- board text added: "r68 65% Board Rev 1.0"
- board text removed: "R60 Standard Board Rev 2.0"
- board text removed: "github.com/rpedde/r60-std"
- board text removed: "http://github.com/rpedde/r60-std"

Commit message: Minor fixes
* fix right arrow that wasn't wired to r4
* change the diode footprint to 0805
Parts:
- D0, D0A1, D0B1, D0C1, D0D1, D0D2, D0D3, D0D4, D0D5, D0D6, D0D7, D0D8, D0D9, D1, D10, D11, D12, D13, D14, D15, D16, D17, D18, D19, D1A1, D1B1, D1C1, D1D1, D2, D20, D21, D22, D23, D24, D25, D26, D27, D28, D29, D2A1, D2B1, D2C1, D3, D30, D31, D32, D33, D34, D35, D36, D37, D38, D39, D3A1, D3B1, D4, D40, D41, D42, D45, D48, D49, D4A1, D5, D6, D7, D8, D9: footprint Diodes_SMD:D_SOD-323 -> Diodes_SMD:D_0805
Connections:
- D0D9 pad 1: (no net) -> /R4
- U1 pad 25: (no net) -> Net-(U1-Pad25)
- U1 pad 32: (no net) -> Net-(U1-Pad32)
- U1 pad 8: (no net) -> Net-(U1-Pad8)
- U1 pad 9: (no net) -> Net-(U1-Pad9)
Routing:
- net /R4: track 315.2 -> 335.3 mm
Other:
- board text added: "r68 65% Board Rev 1.1"
- board text removed: "r68 65% Board Rev 1.0"

Commit message: fix shorted C14
Other:
- board text added: "r68 65% Board Rev 1.2"
- board text removed: "r68 65% Board Rev 1.1"
Changed lines of the file:
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@@
     (links 258)
     (no_connects 0)
-    (area 28.499999 42.787499 333.450001 138.187501)
+    (area 28.424529 41.274999 333.524201 138.261701)
     (thickness 1.6)
     (drawings 16)
@@
     (title r68)
     (date 2017-08-19)
-    (rev 1.1)
+    (rev 1.2)
   )
   (layers
@@
     (effects (font (size 1.5 1.5) (thickness 0.3)) (justify mirror))
   )
-  (gr_text "r68 65% Board Rev 1.1" (at 197.739 126.4285) (layer B.SilkS)
+  (gr_text "r68 65% Board Rev 1.2" (at 197.739 126.4285) (layer B.SilkS)
     (effects (font (size 1.5 1.5) (thickness 0.3)) (justify mirror))
   )
